File: electronics/Servostation_Electronics/Servostation_Electronics.kicad_pcb (KiCad board)
At the start: 2 copper layers, 12 parts, among them J1 Conn_01x05_Female, J2 Conn_01x05_Female, U1 SFH617A-1, U2 SFH617A-1, U3 SFH617A-1, U4 SFH617A-1

Commit message: Edit electronics
Parts:
- D1, D2, D3, D4: footprint LED_THT:LED_D5.0mm -> Diode_THT:D_5W_P5.08mm_Vertical_AnodeUp
- U1, U2, U3, U4: footprint Package_DIP:DIP-4_W7.62mm_SMDSocket_SmallPads -> Package_DIP:DIP-4_W10.16mm_LongPads
- moved R2 111.3 mm to (25.4, 33.0), turned to 0 degrees
- moved J2 106.7 mm to (28.0, 26.1), turned to 0 degrees
- moved R1 96.7 mm to (27.9, 58.4), turned to 0 degrees
- moved U4 95.6 mm to (25.4, 45.7), turned to 90 degrees
- moved D4 89.2 mm to (25.4, 53.3), turned to 180 degrees
- moved U3 78.8 mm to (33.0, 45.7), turned to 90 degrees
- moved D3 69.0 mm to (35.6, 53.3), turned to 180 degrees
- moved U2 62.5 mm to (40.6, 45.7), turned to 90 degrees
- moved J1 50.5 mm to (48.2, 67.8), turned to 180 degrees
- moved D2 48.9 mm to (45.7, 53.3), turned to 180 degrees
- moved U1 44.2 mm to (52.1, 45.7), turned to 90 degrees
- moved D1 29.0 mm to (55.9, 53.3), turned to 180 degrees
Routing:
- net Net-(D1-Pad1): track 87.1 -> 8.13 mm
- net Net-(R2-Pad2): track 51.2 -> 0.00 mm
- net Net-(D1-Pad2): track 27.1 -> 0.00 mm
- net Net-(D4-Pad2): track 27.1 -> 0.00 mm
- net Net-(D2-Pad2): track 25.0 -> 0.00 mm
- net Net-(D3-Pad2): track 25.0 -> 0.00 mm
- net Net-(J2-Pad5): track 15.1 -> 0.00 mm
- net Net-(J2-Pad2): track 14.1 -> 0.00 mm
- net Net-(J2-Pad4): track 13.0 -> 0.00 mm
- net Net-(J1-Pad5): track 13.0 -> 0.00 mm
- net Net-(J2-Pad3): track 12.0 -> 0.00 mm
- net Net-(J2-Pad1): track 12.3 -> 7.94 mm
- net (no net): vias 4 -> 0

Commit message: New electronics
Parts:
- added A1: Arduino_Nano, Module:Arduino_Nano, F.Cu at (125.7, 30.5)
- added J3: Conn_01x05_Male, Connector_PinSocket_2.54mm:PinSocket_1x05_P2.54mm_Vertical, F.Cu at (118.1, 38.1)
- added J4: Conn_01x06_Male, Connector_PinSocket_2.54mm:PinSocket_1x06_P2.54mm_Vertical, F.Cu at (151.8, 48.3)
- added J5: Conn_01x05_Male, Connector_PinSocket_2.54mm:PinSocket_1x05_P2.54mm_Vertical, F.Cu at (113.7, 48.3)
- added J6: Conn_01x03_Female, Connector_Phoenix_MC_HighVoltage:PhoenixContact_MCV_1,5_3-G-5.08_1x03_P5.08mm_Vertical, F.Cu at (159.3, 28.0)
- added R3: R, Resistor_THT:R_Axial_DIN0309_L9.0mm_D3.2mm_P15.24mm_Horizontal, F.Cu at (145.4, 32.4)
- added R4: R, Resistor_THT:R_Axial_DIN0309_L9.0mm_D3.2mm_P15.24mm_Horizontal, F.Cu at (150.5, 42.5)
- moved U2 14.8 mm to (55.2, 48.3)
- moved R1 13.7 mm to (41.3, 61.6)
- moved U1 13.6 mm to (65.4, 48.3)
- moved D1 13.3 mm to (69.2, 53.3)
- moved D2 13.3 mm to (59.0, 53.3)
- moved D4 13.3 mm to (38.7, 53.3)
- moved J1 13.3 mm to (61.6, 67.8)
- moved R2 13.3 mm to (38.7, 33.0)
- moved J2 13.3 mm to (41.3, 26.1)
- moved D3 13.3 mm to (48.9, 53.3)
- moved U3 12.2 mm to (45.1, 47.6)
- moved U4 9.70 mm to (34.9, 47.6)
Routing:
- net GND: track 0.00 -> 146.7 mm
- net +5V: track 0.00 -> 125.7 mm
- net Net-(D1-Pad1): track 8.13 -> 72.8 mm
- net Net-(R2-Pad2): track 0.00 -> 45.6 mm
- net Net-(D4-Pad2): track 0.00 -> 29.2 mm
- net Net-(D3-Pad2): track 0.00 -> 23.7 mm
- net Net-(D2-Pad2): track 0.00 -> 21.1 mm
- net Net-(D1-Pad2): track 0.00 -> 20.9 mm
- net AN_INPUT: track 0.00 -> 16.2 mm
- net Net-(J2-Pad2): track 0.00 -> 15.9 mm
- net Net-(J2-Pad5): track 0.00 -> 14.9 mm
- net Net-(J6-Pad2): track 0.00 -> 14.1 mm
- net Net-(J2-Pad4): track 0.00 -> 12.8 mm
- net Net-(J2-Pad3): track 0.00 -> 12.6 mm
- net Net-(A1-Pad9): track 0.00 -> 12.1 mm
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
Commit message: software and electronics update
Parts:
- added D5: LED, Diode_THT:D_5W_P5.08mm_Vertical_AnodeUp, F.Cu at (113.0, 37.1)
- added J10: Conn_01x03_Male, Connector:FanPinHeader_1x03_P2.54mm_Vertical, F.Cu at (241.7, 40.2)
- added J11: Conn_01x03_Male, Connector:FanPinHeader_1x03_P2.54mm_Vertical, F.Cu at (242.6, 52.0)
- added J12: Conn_01x03_Male, Connector_PinHeader_2.54mm:PinHeader_1x03_P2.54mm_Vertical, F.Cu at (247.6, 44.0)
- added J6: Conn_01x03_Male, Connector_PinHeader_2.54mm:PinHeader_1x03_P2.54mm_Vertical, F.Cu at (224.8, 49.1)
- added J8: Conn_01x03_Male, Connector:FanPinHeader_1x03_P2.54mm_Vertical, F.Cu at (230.8, 53.0)
- added J9: Conn_01x03_Male, Connector:FanPinHeader_1x03_P2.54mm_Vertical, F.Cu at (229.8, 41.1)
- added R5: R, Resistor_THT:R_Axial_DIN0309_L9.0mm_D3.2mm_P5.08mm_Vertical, F.Cu at (120.7, 66.4)
- renumbered J5 to J3, J3 to J4, J4 to J5, J6 to J7
Connections:
- A1 pad 13: unconnected-(A1-Pad13) -> Net-(A1-Pad13)
- J4 pad 1: +5V -> GND
Routing:
- net Net-(J10-Pad1): track 0.00 -> 53.1 mm
- net GND: track 146.7 -> 104.5 mm
- net Net-(D5-Pad2): track 0.00 -> 36.8 mm
- net Net-(J10-Pad3): track 0.00 -> 33.9 mm
- net Net-(J6-Pad2): track 0.00 -> 17.7 mm
- net Net-(J11-Pad2): track 0.00 -> 11.3 mm
- net Net-(A1-Pad13): track 0.00 -> 9.82 mm
- net Net-(J6-Pad3): track 0.00 -> 9.80 mm
- net Net-(J10-Pad2): track 0.00 -> 6.51 mm
- net (no net): vias 8 -> 12
- added copper zone on F.Cu, net (none)
Other:
- board text added: "Arduino Board"
- board text added: "Opto-Isolator Board"
- board text added: "Servo-Connector Board"
